Commit message: Add robot localization

File: gem_simulator_modified/urdf/gem.urdf.xacro (robot description, xacro)
@@ -70,5 +70,5 @@
   </joint>
   <joint name="center_link" type="fixed">
-    <origin xyz="0.87 0 0.151" rpy="0 0 0"/>
+    <origin xyz="0.0 0 0.0" rpy="0 0 0"/>
     <parent link="base_link"/>
     <child link="center_link"/>

Commit message: Add path tracking mpc

File: gem_simulator_modified/urdf/gem.urdf.xacro (robot description, xacro)
@@ -70,5 +70,5 @@
   </joint>
   <joint name="center_link" type="fixed">
-    <origin xyz="0.0 0 0.0" rpy="0 0 0"/>
+    <origin xyz="0.87 0 0.0" rpy="0 0 0"/>
     <parent link="base_link"/>
     <child link="center_link"/>

Commit message: Add costmap subscriber

File: gem_simulator_modified/urdf/gem.urdf.xacro (robot description, xacro)
@@ -24,4 +24,6 @@
   <link name="base_link">
   </link>
+  <link name="center_footprint">
+  </link>
   <link name="center_link">
     <inertial>
@@ -73,4 +75,9 @@
     <parent link="base_link"/>
     <child link="center_link"/>
+  </joint>
+  <joint name="center_footprint_joint" type="fixed">
+    <origin xyz="0.0 0 -0.44" rpy="0 0 0"/>
+    <parent link="center_link"/>
+    <child link="center_footprint"/>
   </joint>
   <!-- ******************************************* Fixed links below ******************************************* -->

Commit message: Add centered base_footprint

File: gem_simulator_modified/urdf/gem.urdf.xacro (robot description, xacro)
@@ -24,6 +24,4 @@
   <link name="base_link">
   </link>
-  <link name="center_footprint">
-  </link>
   <link name="center_link">
     <inertial>
@@ -72,12 +70,7 @@
   </joint>
   <joint name="center_link" type="fixed">
-    <origin xyz="0.87 0 0.0" rpy="0 0 0"/>
+    <origin xyz="0 0 0" rpy="0 0 0"/>
     <parent link="base_link"/>
     <child link="center_link"/>
-  </joint>
-  <joint name="center_footprint_joint" type="fixed">
-    <origin xyz="0.0 0 -0.44" rpy="0 0 0"/>
-    <parent link="center_link"/>
-    <child link="center_footprint"/>
   </joint>
   <!-- ******************************************* Fixed links below ******************************************* -->

Commit message: Add theta term to obj function

File: gem_simulator_modified/urdf/gem.urdf.xacro (robot description, xacro)
@@ -1,5 +1,5 @@
 <?xml version="1.0"?>
 <robot name="gem" xmlns:xacro="http://www.ros.org/wiki/xacro">
-  <xacro:property name="steer_angle" value="0.61"/>
+  <xacro:property name="steer_angle" value="0.78"/>
   <xacro:property name="PI" value="3.1415926835897931"/>
   <xacro:property name="tyre_length" value="0.16"/>
